File: WU-MSNS6101HT.sch (KiCad schematic (older format))
At the start: 31 parts, among them J1 Conn_01x04, J2 Conn_01x04, Q1 AO3400A, Q2 AO3400A, U1 MPU-6050, U2 LMV358, U3 74AHC1G08

Commit message: Add a pull down res for
Parts:
- added R16: 10k, Resistor_SMD:R_0805_2012Metric_Pad1.15x1.40mm_HandSolder, symbol Device:R
- R1: value 1k -> 4.7k
Connections:
- net GND: now also R16.2
- net HTPWM: now also R16.1
Other:
- moved on the sheet: J2
Changed lines of the file:
@@
 EESchema Schematic File Version 4
-LIBS:WU-MSNS601HT-cache
+LIBS:WU-MSNS6101HT-cache
 EELAYER 29 0
 EELAYER END
@@
 P 2200 2500
 F 0 "R1" H 2270 2546 50  0000 L CNN
-F 1 "1k" H 2270 2455 50  0000 L CNN
+F 1 "4.7k" H 2270 2455 50  0000 L CNN
 F 2 "Resistor_SMD:R_0805_2012Metric_Pad1.15x1.40mm_HandSolder" V 2130 2500 50  0001 C CNN
 F 3 "~" H 2200 2500 50  0001 C CNN
@@
 L Connector_Generic:Conn_01x04 J2
 U 1 1 5D6E9950
-P 7500 4900
-F 0 "J2" H 7580 4892 50  0000 L CNN
-F 1 "Conn_01x04" H 7580 4801 50  0000 L CNN
-F 2 "Connector_PinSocket_2.54mm:PinSocket_1x04_P2.54mm_Vertical" H 7500 4900 50  0001 C CNN
-F 3 "~" H 7500 4900 50  0001 C CNN
-	1    7500 4900
+P 7500 4200
+F 0 "J2" H 7580 4192 50  0000 L CNN
+F 1 "Conn_01x04" H 7580 4101 50  0000 L CNN
+F 2 "Connector_PinSocket_2.54mm:PinSocket_1x04_P2.54mm_Vertical" H 7500 4200 50  0001 C CNN
+F 3 "~" H 7500 4200 50  0001 C CNN
+	1    7500 4200
 	1    0    0    -1
 $EndComp
@@
 L power:+3.3V #PWR027
 U 1 1 5D6EEDB6
-P 7200 4750
-F 0 "#PWR027" H 7200 4600 50  0001 C CNN
-F 1 "+3.3V" H 7215 4923 50  0000 C CNN
-F 2 "" H 7200 4750 50  0001 C CNN
-F 3 "" H 7200 4750 50  0001 C CNN
-	1    7200 4750
+P 7200 4050
+F 0 "#PWR027" H 7200 3900 50  0001 C CNN
+F 1 "+3.3V" H 7215 4223 50  0000 C CNN
+F 2 "" H 7200 4050 50  0001 C CNN
+F 3 "" H 7200 4050 50  0001 C CNN
+	1    7200 4050
 	1    0    0    -1
 $EndComp
@@
 L power:+5V #PWR026
 U 1 1 5D6EF6E6
-P 6950 4750
-F 0 "#PWR026" H 6950 4600 50  0001 C CNN
-F 1 "+5V" H 6965 4923 50  0000 C CNN
-F 2 "" H 6950 4750 50  0001 C CNN
-F 3 "" H 6950 4750 50  0001 C CNN
-	1    6950 4750
+P 6950 4050
+F 0 "#PWR026" H 6950 3900 50  0001 C CNN
+F 1 "+5V" H 6965 4223 50  0000 C CNN
+F 2 "" H 6950 4050 50  0001 C CNN
+F 3 "" H 6950 4050 50  0001 C CNN
+	1    6950 4050
 	1    0    0    -1
 $EndComp
@@
 L power:GNDREF #PWR028
 U 1 1 5D6F069A
-P 7200 5200
-F 0 "#PWR028" H 7200 4950 50  0001 C CNN
-F 1 "GNDREF" H 7205 5027 50  0000 C CNN
-F 2 "" H 7200 5200 50  0001 C CNN
-F 3 "" H 7200 5200 50  0001 C CNN
-	1    7200 5200
-	1    0    0    -1
-$EndComp
-Wire Wire Line
-	7300 4900 6950 4900
-Wire Wire Line
-	6950 4900 6950 4750
-Wire Wire Line
-	7300 4800 7200 4800
-Wire Wire Line
-	7200 4800 7200 4750
-Wire Wire Line
-	7300 5100 7200 5100
-Wire Wire Line
-	7200 5100 7200 5200
-Text GLabel 7000 5000 0    50   Input ~ 0
+P 7200 4500
+F 0 "#PWR028" H 7200 4250 50  0001 C CNN
+F 1 "GNDREF" H 7205 4327 50  0000 C CNN
+F 2 "" H 7200 4500 50  0001 C CNN
+F 3 "" H 7200 4500 50  0001 C CNN
+	1    7200 4500
+	1    0    0    -1
+$EndComp
+Wire Wire Line
+	7300 4200 6950 4200
+Wire Wire Line
+	6950 4200 6950 4050
+Wire Wire Line
+	7300 4100 7200 4100
+Wire Wire Line
+	7200 4100 7200 4050
+Wire Wire Line
+	7300 4400 7200 4400
+Wire Wire Line
+	7200 4400 7200 4500
+Text GLabel 7000 4300 0    50   Input ~ 0
 HTPWM
 Wire Wire Line
-	7300 5000 7000 5000
+	7300 4300 7000 4300
 NoConn ~ 6300 2550
 Wire Notes Line
@@
 Wire Notes Line
 	6650 500  6650 6600
+Text GLabel 7000 5000 0    50   Input ~ 0
+HTPWM
+$Comp
+L Device:R R16
+U 1 1 5D611E10
+P 7200 5300
+F 0 "R16" H 7270 5346 50  0000 L CNN
+F 1 "10k" H 7270 5255 50  0000 L CNN
+F 2 "Resistor_SMD:R_0805_2012Metric_Pad1.15x1.40mm_HandSolder" V 7130 5300 50  0001 C CNN
+F 3 "~" H 7200 5300 50  0001 C CNN
+	1    7200 5300
+	1    0    0    -1
+$EndComp
+$Comp
+L power:GNDREF #PWR029
+U 1 1 5D612863
+P 7200 5600
+F 0 "#PWR029" H 7200 5350 50  0001 C CNN
+F 1 "GNDREF" H 7205 5427 50  0000 C CNN
+F 2 "" H 7200 5600 50  0001 C CNN
+F 3 "" H 7200 5600 50  0001 C CNN
+	1    7200 5600
+	1    0    0    -1
+$EndComp
+Wire Wire Line
+	7200 5150 7200 5000
+Wire Wire Line
+	7200 5000 7000 5000
+Wire Wire Line
+	7200 5450 7200 5600
 $EndSCHEMATC
