File: WU-MSNS6101HT.kicad_pcb (KiCad board)
At the start: 2 copper layers, 30 x 30 mm, 31 parts, among them J1 Conn_01x04, J2 Conn_01x04, Q1 AO3400A, Q2 AO3400A, U1 MPU-6050, U2 LMV358, U3 74AHC1G08

Commit message: Rework the PCB
Parts:
- added R16: 10k, Resistor_SMD:R_0805_2012Metric_Pad1.15x1.40mm_HandSolder, F.Cu at (62.7, 122.4)
- R1: value 1k -> 4.7k
- TH1: footprint digikey-footprints:Terminal_Block_D1.3mm_P5mm -> Connector_PinHeader_2.54mm:PinHeader_1x02_P2.54mm_Vertical
- moved TH1 2.03 mm to (70.2, 114.8), turned to 180 degrees
Routing:
- net HTPWM: track 6.83 -> 13.3 mm
- net +5V: track 14.5 -> 16.1 mm
- net +3V3: track 75.1 -> 74.3 mm
